File: board/buck-converter.sch (EAGLE design)
At the start: 8 parts, among them Q1 MOSFET-PCHANNELSMD, U1 Tiny85-20-SMT

Commit message: Not sure what these changes are
Parts:
- added C3: 47uF, SparkFun-Capacitors:47UF-50V-20%(ELECT)
- added L2: 180uH, SparkFun-Passives:INDUCTORCR54
- added Q2: 2N3904, SparkFun-DiscreteSemi:TRANSISTOR_NPNBC547
- added R3, R4: 10k, SparkFun-Resistors:RESISTOR0603
- added R5: 820, SparkFun-Resistors:RESISTOR0603
- C1: value (none) -> 100uF
- C2: value (none) -> 47uF
- L1: value (none) -> 180uH
- Q1: value MOSFET-PCHANNELSMD -> P-CHANNEL
- R1: value (none) -> 30k
- R2: value (none) -> 15k
Connections:
- new net FB: R1.1, R2.2
- new net N$2: Q1.G, Q2.C, R3.1
- new net N$3: L1.1, Q1.D
- new net N$4: D1.A, L1.2
- new net N$5: C2.+, D1.C, L2.1
- new net N$8: Q2.B, R4.2, R5.1
- new net PWM: R5.2, U1.PB4(ADC2)
- new net VOUT: C3.+, L2.2, R1.2
- new net V_BATT: C1.+, Q1.S, R3.2
- net GND: now also C1.-, C2.-, C3.-, Q2.E, R2.1, R4.1
Other:
- note added: "VDiv 1.1v"
- note added: "VOUT is 3.3v"
- moved on the sheet: C1, C2, D1, L1, Q1, R1, R2
